File: G3 Personality Card USB.kicad_sch (KiCad schematic)
At the start: 68 parts, among them J1 USB_A, Q7 MMBT3906, Q8 MMBT3906, Q9 MMBT3906, U1 LTC1865-S8, U6 CMD-USB0670, U9 LTC1865-S8

Commit message: Add files via upload
Parts:
- removed L26: FB, symbol Device:L_Ferrite_Small
- added C92, C96: 0.1uF, symbol Device:C_Small
- C106: value 110nF -> 0.1uF
- C114: value 100nF -> 0.1uF
- renumbered J1 to J11
Connections:
- net at R43.1: now also C110.1, LP1.8, R61.1; no longer U6.13 (VD1+)
- net at C99.2, D2.1 (K), U6.12 (VDD3)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: now also C96.2
- net at U6.7 (VDD): now also C92.2
- net at U6.8 (VSS): now also C96.1
- new net: R43.2, U6.13 (VD1+)
- no-connect marks 9 -> 10
Other:
- note added: "Power Connection with Fuse"
- note added: "Power Connection with Glue Logic Values not known Not needed when employing a fuse"
- note added: "Startup Circuit Values not known"
- moved on the sheet: C106, C109, C110, C116, C118, C122, C124, C129, C131, C157, D1, F1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
