File: G3 Personality Card USB.kicad_sch (KiCad schematic)
At the start: 69 parts, among them J11 USB_A, Q7 MMBT3906, Q8 MMBT3906, Q9 MMBT3906, U1 LTC1865-S8, U6 CMD-USB0670, U9 LTC1865-S8

Commit message: Add files via upload
Other:
- company: Schematic created by croissantking on the 68kmla forums, with invaluable help from phipli -> Schematic created by @croissantking on the 68kMLA forums with invaluable help from @phipli
Changed lines of the file:
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@@
     (date "2023-07-12")
     (rev "2")
-    (company "Schematic created by croissantking on the 68kmla forums, with invaluable help from phipli")
+    (company "Schematic created by @croissantking on the 68kMLA forums with invaluable help from @phipli")
   )
   (junction (at 190.5 152.4) (diameter 0) (color 0 0 0 0)

Commit message: Add files via upload
Other:
- company: Schematic created by @croissantking on the 68kMLA forums with invaluable help from @phipli -> Schematic by @croissantking on the 68kMLA forums with invaluable help from @phipli
Changed lines of the file:
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@@
     (date "2023-07-12")
     (rev "2")
-    (company "Schematic created by @croissantking on the 68kMLA forums with invaluable help from @phipli")
+    (company "Schematic by @croissantking on the 68kMLA forums with invaluable help from @phipli")
   )
   (junction (at 190.5 152.4) (diameter 0) (color 0 0 0 0)
@@
       (effects (font (size 1.27 1.27) italic) hide)
     )
-    (property "Datasheet" "http://www.ti.com/lit/ds/symlink/lm3s6911.pdf" (at -25.4 64.77 90)
+    (property "Datasheet" "http://www.bitsavers.org/components/cmd/MAN-000670-000_USB0670_673_PCI-USB_ASIC_Rev_1.8_199903.pdf" (at -25.4 64.77 90)
       (effects (font (size 0 0)) hide)
     )
