File: Whisper/Whisper USB V4.kicad_sch (KiCad schematic)
At the start: 69 parts, among them J11 USB_A, Q7 PMBT3906, Q8 MMBT3904L, Q9 MMBT3904L, U1 LM393, U6 CMD 0670B-400 / OPTi FireLink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, U9 UCC3912

Commit message: Add files via upload
Parts:
- renumbered U1 to U20
Changed lines of the file:
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@@
   (netclass_flag "" (length 2.54) (shape round) (at 162.56 175.26 180)
     (effects (font (size 1.27 1.27)) (justify right bottom))
-    (property "Netclass" "PERCH #178/VDD" (at 156.21 180.34 0)
+    (property "Netclass" "PERCH #178/+5VSB" (at 154.94 180.34 0)
       (effects (font (size 1 1) italic) (justify left))
     )
@@
   (symbol (lib_id "Analog_ADC:LM393") (at 243.84 151.13 270) (unit 1)
     (in_bom yes) (on_board yes) (dnp no)
-    (property "Reference" "U1" (at 248.92 153.67 90)
+    (property "Reference" "U20" (at 248.92 153.67 90)
       (effects (font (size 1.27 1.27)))
     )
@@
       (project "G3 Whisper Card USB"
         (path "/f6767184-bfed-4427-86eb-57243872235b"
-          (reference "U1") (unit 1)
-        )
-      )
+          (reference "U20") (unit 1)
+        )
+      )
